Commit message: PointClouds using Laser_Assembler

File: urdf/DataLogger.urdf (robot description, URDF)
Before this commit: robot DataLogger, 2 links, 1 joints
Links:
- link camera: geometry visual mesh filename=package://div_datalogger_postprocess/meshes/Camera.stl scale=0.01 0.01 0.01
- link laser: geometry visual mesh filename=package://div_datalogger_postprocess/meshes/Lidar_Imu.stl scale=0.01 0.01 0.01

Commit message: update to reference frames

File: urdf/DataLogger.urdf (robot description, URDF)
Before this commit: robot DataLogger, 2 links, 1 joints
Joints:
- joint laser_to_camera: origin xyz=0 0.046 -0.093 -> xyz=0 0 -0.117

Commit message: model frames change - calibration needed laser-imu

File: urdf/DataLogger.urdf (robot description, URDF)
Before this commit: robot DataLogger, 2 links, 1 joints
Links:
- removed link camera
- added link base_link; visual mesh filename=package://div_datalogger_postprocess/meshes/DataLogger_ImuF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 scale=0.01 0.01 0.01
- link laser: geometry visual cylinder length=0.06 radius=0.02
Joints:
- joint laser_to_camera: child camera -> laser; origin xyz=0 0 -0.117 -> xyz=0 0 -0.1004 rpy=3.08 0 3.14; parent laser -> base_link

Commit message: calibration of axis orientation

File: urdf/DataLogger.urdf (robot description, URDF)
Before this commit: robot DataLogger, 2 links, 1 joints
Joints:
- joint laser_to_camera: origin xyz=0 0 -0.1004 rpy=3.08 0 3.14 -> xyz=0 0 -0.1004 rpy=3.14 0.008 3.14

Commit message: node for gyro-drift correction, launch file for gyro correction, postprocess.launch updated

File: urdf/DataLogger.urdf (robot description, URDF)
Before this commit: robot DataLogger, 2 links, 1 joints
Links:
- removed link base_link
- added link base_link_corrected; visual mesh filename=package://div_datalogger_postprocess/meshes/DataLogger_ImuF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 scale=0.01 0.01 0.01
Joints:
- joint laser_to_camera: origin xyz=0 0 -0.1004 rpy=3.08 0 3.14 -> xyz=0 0 -0.1004 rpy=3.045 -0.01 3.14; parent base_link -> base_link_corrected
