Commit message: implementation of hector_mapping:  trial

File: urdf/DataLogger_v2.urdf (robot description, URDF)
Before this commit: robot DataLogger, 2 links, 1 joints
Joints:
- joint laser_to_camera: origin xyz=0 0 -0.1004 rpy=3.14 0 3.14 -> xyz=0 0 -0.1004 rpy=3.08 0.1 3.14

Commit message: lateral clearance extraction using box filter and clustering

File: urdf/DataLogger_v2.urdf (robot description, URDF)
Before this commit: robot DataLogger, 2 links, 1 joints
Joints:
- joint laser_to_camera: origin xyz=0 0 -0.1004 rpy=3.08 0.1 3.14 -> xyz=0 0 -0.1004 rpy=3.075 0.095 3.14
